File: circuits-v0.2/hex-minidrive.kicad_pcb (KiCad board)
At the start: 4 copper layers, 29 x 51 mm, 97 parts, among them X1 16MHz

Commit message: Order v0.2 circuits.
Parts:
- turned Q3 to 0 degrees
- turned Q5 to 0 degrees
- turned Q7 to -90 degrees
- turned D2 to -90 degrees
- turned Q1 to 0 degrees
- turned Q2 to 180 degrees
- turned Q4 to 180 degrees
- turned Q6 to 180 degrees
- turned Q8 to 90 degrees
- turned U1 to -90 degrees
- turned U3 to 90 degrees
- turned U4 to 180 degrees
- turned U5 to 180 degrees
- turned U6 to 180 degrees
- turned U8 to -90 degrees
