File: circuits-v0.3/hex-minidrive.kicad_sch (KiCad schematic)
At the start: 81 parts, among them X1 16MHz

Commit message: Fix positioning errors and realize SPI3 is not in the bootloader options.
Parts:
- Q1, Q3, Q5, Q7: footprint Library:DFN-8_L3.0-W3.0-P0.65-BL-MOSFET -> Library:DFN-8_L3.0-W3.0-P0.65-BL-MOSFET_shifted

Commit message: Sigh, SPI3 cannot be used for the bootloader, move to SPI2. Finish v0.3 again.
Connections:
- net I2C2_SCL: now also U1.43 (PA9); no longer U1.22 (PC4)
- net TIM1_CH2: now also U1.9 (PC1); no longer U1.43 (PA9)
- net TIM1_CH2N: now also U1.46 (PA12); no longer U1.36 (PB14)
- net TIM1_CH3: now also U1.10 (PC2); no longer U1.44 (PA10)
- net ADC1_IN4/M3_CURRENT: now reaches U1.17 (PA3)
- net ADC1_IN4/M3_CURRENT: now also U2.13 (OUT3)
- net ADC2_IN17/M4_CURRENT: now reaches U1.18 (PA4)
- net ADC2_IN17/M4_CURRENT: now also U2.19 (OUT4)
- net SPI2_NSS: now reaches U1.34 (PB12)
- net SPI2_NSS: now also FPC1.8
- net SPI2_SCK: now reaches U1.35 (PB13)
- net SPI2_SCK: now also FPC1.7
- net ADC1_IN12/M3_CURRENT: no longer names the net of U1.25 (PB1)
- net ADC1_IN12/M3_CURRENT: no longer U2.13 (OUT3)
- net ADC2_IN14/M4_CURRENT renamed ADC2_IN14/VOLTAGE
- net ADC2_IN14/VOLTAGE: now also C115.2, R18.1, R19.2; no longer U2.19 (OUT4)
- removed net ADC2_IN15/VOLTAGE: C115.2, R18.1, R19.2, U1.37 (PB15)
- net SPI3_MISO: no longer names the net of U1.57 (PB4)
- net SPI3_MISO: no longer FPC1.6
- net SPI3_MOSI: no longer names the net of U1.54 (PC12)
- net SPI3_MOSI: no longer FPC1.5
- net SPI3_NSS: no longer names the net of U1.51 (PA15)
- net SPI3_NSS: no longer FPC1.8
- net SPI3_SCK renamed TIM2_CH2/BLUE_LED
- net TIM2_CH2/BLUE_LED: now also R16.2; no longer FPC1.7
- net TIM2_CH3/BLUE_LED: no longer names the net of U1.30 (PB10)
- net TIM2_CH3/BLUE_LED: no longer R16.2
- new net SPI2_MISO: FPC1.6, U1.36 (PB14)
- new net SPI2_MOSI: FPC1.5, U1.37 (PB15)
