File: circuits-v0.4/hex-minidrive.kicad_sch (KiCad schematic)
At the start: 81 parts, among them X1 16MHz

Commit message: Convert to kicad 10.
Parts:
- FPC1, FPC2, FPC3, LED1, Q1, Q2, Q3, Q4, Q5, Q6, Q7, Q8, U1, U2, U3, U4, U5, U6: value ~ -> (none)
Changed lines of the file:
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@@
 (kicad_sch
-	(version 20250114)
+	(version 20260306)
 	(generator "eeschema")
-	(generator_version "9.0")
+	(generator_version "10.0")
 	(paper "A2")
 	(title_block

Commit message: Begin the v0.4 driver code.
Parts:
- added R14: 10kΩ, Library:R0402, symbol Library:0402WGF1002TCE Resistor 10kΩ
Connections:
- net 3V3: now also R14.1
- net 3V3A: now also R13.2
- net NRST: now also R14.2
- net VREF: no longer R13.2
Other:
- note added: "Add pull-up to 3V3 to ensure it's stable."
- note added: "Hex Mini Driver This is a quad output, motor driver for stepper, brushless or 2 DC motors. The board comes provisioned with 2 I2C connectors for plug in rotation sensors AS5600 (preferably the Hex mini flex rotation sensor). Target limits are 6-30V supply range and 5A of current. TODO for this version: [v] Remember to deal with the STM32 voltage reference, needs to be isolated from the amplifier.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"
- note added: "Leave VREF unconnected except the caps."
- note removed: "Hex Mini Driver This is a quad output, motor driver for stepper, brushless or 2 DC motors. The board comes provisioned with 2 I2C connectors for plug in rotation sensors AS5600 (preferably the Hex mini flex rotation sensor). Target limits are 6-30V supply range and 5A of current. TODO for this version: [v] Swap components to 0402 where possible, 0603 where not. [v] Optimize for 2 sided tiny circu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"
- moved on the sheet: C103, C104, C107, C108, C110, R12, R13, X1

Commit message: Make schematic for v0.4 driver circuit.
Parts:
- removed C41: 10uF, Library:C1206, symbol Library:CL31A106KBHNNNE Capacitor 10uF
- removed C42, C43: 100nF, Library:C0603, symbol Library:CC0603KRX7R9BB104 Capacitor 100nF
- removed C44, C45: 22uF, Library:C0805, symbol Library:CL21A226MAQNNNE Capacitor 22uF
- removed C46: 100pF, Library:C0402, symbol Library:0402CG101J500NT Capacitor 100pF
- removed FPC1: (no value), Library:FPC-SMD_20P-P0.50_XUNPU_FPC-05F-20PH20, symbol Library:FPC-05F-20PH20 Connector 6P 0.5mm spacing FPC
- removed L1: 15uH, Library:IND-SMD_L4.0-W4.0, symbol Library:FHD4020S-150MT 15uH inductor
- removed R41: 49.9Ω, Library:R0402, symbol Library:0402WGF499JTCE Resistor 49.9Ω
- removed R42: 100kΩ, Library:R0402, symbol Library:0402WGF1003TCE Resistor 100kΩ
- removed R43: 13.3kΩ, Library:R0402, symbol Library:FRC0402F1332TS Resistor 13.3kΩ
- removed U4: (no value), Library:SOT-23-6_L2.9-W1.6-P0.95-LS2.8-BL, symbol Library:TPS54202DDCR Buck converter
- added D1: ~, Library:SOD-123_L2.7-W1.6-LS3.7-RD-1, symbol Library:B5819W_C8598 Schottky diode
- added D2, D3: ~, Library:SOT-23-3_L3.0-W1.7-P0.95-LS2.9-BR, symbol Library:PSM712-LF-T7 ETV/ESD Diodes
- added FPC1: (no value), Library:FPC-SMD_20P-P0.50_XUNPU_FPC-05F-20PH20, symbol Library:FPC-05F-20PH20 Connector 20P 0.5mm spacing FPC
- added H2, H3: 2P-1.27mm-header, Library:HDR-TH_2P-P1.27-V-M-2, symbol Library:ZX-PZ1.27-1-2PZZ Connector 2P 1.27mm spacing
- added L3: 300mΩ, Library:L0805, symbol Library:GZ2012D601TF Ferrite bead
- added R5, R6: 5.1kΩ, Library:R0402, symbol Library:0402WGF5101TCE Resistor 5.1kΩ
- added USB1: ~, Library:USB-C-SMD_TYPE-C16PIN, symbol Library:TYPE-C16PIN USB connector
Connections:
- net SPI2_MISO is gone; now on net TIM1_CH2N: U1.36 (PB14)
- net 5V: now also D1.1 (-)
- net BOOT0/STOP: now also D3.2 (A1), USB1.B8 (SBU2)
- net GND: now also D2.3 (K), D3.3 (K), FPC1.11, FPC1.12, FPC1.13, FPC1.14, FPC1.15, FPC1.16, FPC1.17, FPC1.18, FPC1.19, FPC1.20, H2.1, H2.2, R5.1, R6.1, USB1.A1B12 (GND), USB1.B1A12 (GND)
- net NRST: now also D3.1 (A1), USB1.A8 (SBU1)
- net TIM1_CH2N: no longer U1.46 (PA12)
- net TIM2_CH2/BLUE_LED: now also U1.13 (PA1); no longer U1.56 (PB3)
- net USART3_RX: no longer U1.53 (PC11)
- net USART3_TX: no longer U1.52 (PC10)
- net VCC: now also FPC1.1, FPC1.10, FPC1.2, FPC1.3, FPC1.4, FPC1.5, FPC1.6, FPC1.7, FPC1.8, FPC1.9, H3.1, H3.2
- net TIM2_CH1/RED_LED: now reaches U1.19 (PA5)
- net TIM2_CH1/RED_LED: now also R17.1
- net TIM2_CH3/GREEN_LED: now reaches U1.30 (PB10)
- net TIM2_CH3/GREEN_LED: now also R15.2
- net USB_D_N: now reaches U1.45 (PA11)
- net USB_D_N: now also D2.1 (A1), USB1.A7 (DN1), USB1.B7 (DN2)
- net SPI2_MOSI: no longer names the net of U1.37 (PB15)
- net SPI2_NSS: no longer names the net of U1.34 (PB12)
- net SPI2_SCK: no longer names the net of U1.35 (PB13)
- net TIM4_CH1/RED_LED: no longer names the net of U1.59 (PB6)
- net TIM4_CH1/RED_LED: no longer R17.1
- net TIM4_CH2/GREEN_LED: no longer names the net of U1.60 (PB7)
- net TIM4_CH2/GREEN_LED: no longer R15.2
- new net USB:5V: L3.1, USB1.A4B9 (VBUS), USB1.B4A9 (VBUS)
- new net USB:5V-filtered: D1.2 (+), L3.2
- new net USB:CC1: R6.2, USB1.A5 (CC1)
- new net USB:CC2: R5.2, USB1.B5 (CC2)
- new net USB_D_P: D2.2 (A1), U1.46 (PA12), USB1.A6 (DP1), USB1.B6 (DP2)
- no-connect marks 32 -> 41
Other:
- note added: "Elestrostatic discharge protection"
- note added: "Eusebiu - USB C"
- note added: "Ferrite bead filtering 5V USB line."
- note added: "Input voltage measurement"
- note added: "Note: pullup resistor is included in STM32G4 series."
- note added: "Power FPC connector"
- note added: "SBU1 and SBU2 are coonected to Reset and Boot0 pins so we can flash new software over USB with the builtin bootloader, let's see if it works."
- note removed: "Has internal pullup to enable"
- note removed: "Input power step down to 5V:"
- note removed: "Power and control, FPC connector"
- moved on the sheet: C0, C1, C101, C102, C107, C108, C115, C2, C21, C3, C31, C32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

Commit message: Almost done re-wiring v0.4
Connections:
- net +Probe-1: now also U2.6 (IN+2); no longer U2.4 (IN+1)
- net +Probe-2: now also U2.4 (IN+1); no longer U2.6 (IN+2)
- net -Probe-1: now also U2.7 (IN±2); no longer U2.3 (IN±1)
- net -Probe-2: now also U2.3 (IN±1); no longer U2.7 (IN±2)
- net ADC1_IN1/M1_CURRENT: now also U2.8 (OUT2); no longer U2.2 (OUT1)
- net ADC2_IN3/M2_CURRENT: now also U2.2 (OUT1); no longer U2.8 (OUT2)
- net TIM2_CH1/RED_LED renamed TIM2_CH1/GREEN_LED
- net TIM2_CH1/GREEN_LED: now also R15.2; no longer R17.1
- net TIM2_CH3/GREEN_LED renamed TIM2_CH3/RED_LED
- net TIM2_CH3/RED_LED: now also R17.1; no longer R15.2

Commit message: Tentatively done wiring v0.4.
Parts:
- removed C4, C6: 10uF, Library:C1206, symbol Library:CL31A106KBHNNNE Capacitor 10uF
- renumbered C5 to C4
Other:
- moved on the sheet: C4

Commit message: Finish and generate production files for v0.4 driver circuit.
Parts:
- H2, H3: now not fitted
- Q1, Q3, Q5, Q7: FT Origin (none) -> Anchor
Other:
- note added: "Hex Mini Driver This is a quad output, motor driver for stepper, brushless or 2 DC motors. The board comes provisioned with 2 I2C connectors for plug in rotation sensors AS5600 (preferably the Hex mini flex rotation sensor). Target limits are 6-30V supply range and 5A of current."
- note removed: "Hex Mini Driver This is a quad output, motor driver for stepper, brushless or 2 DC motors. The board comes provisioned with 2 I2C connectors for plug in rotation sensors AS5600 (preferably the Hex mini flex rotation sensor). Target limits are 6-30V supply range and 5A of current. TODO for this version: [v] Remember to deal with the STM32 voltage reference, needs to be isolated from the amplifier.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"
Changed lines of the file:
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@@
 	(title_block
 		(title "Hex mini servo driver")
-		(rev "version 0.3")
+		(date "2026-06-03")
+		(rev "version 0.4")
 		(company "Hex Robotics Limited")
 		(comment 1 "Author: Calin Mocanu")
