File: master-circuit-v0.2/back-to-back-mosfets.kicad_sch (KiCad schematic)
At the start: 6 parts

Commit message: Convert to kicad 10.
Parts:
- Q1, Q2, U2: value ~ -> (none)

Commit message: Working on new circuit.
Other:
- moved on the sheet: Q1
