File: master-circuit-v0.2/master-circuit.kicad_sch (KiCad schematic)
At the start: 128 parts, among them U6 20nF 5%, X2 24MHz

Commit message: Argh, some chips out of stock, got to do a slight redesign.
Parts:
- removed C19: 1uF, Library:C0603, symbol Library:CL10A105KB8NNNC Capacitor 1uF
- removed D13, D15, D3: (no value), Library:SOD-123_L2.7-W1.6-LS3.7-RD-1, symbol Library:B5819W_C8598 Schottky diode
- removed U5: (no value), Library:TDFN-6_L2.0-W2.0-P0.65-TL-EP, symbol Library:HUSB237-AA001-DN06R USB Power receiver controller
- removed U6: 20nF 5%, Library:C0805, symbol Library:CC0805JRX7R9BB203 Capacitor 20nF 5%
- added C29, C55, C56: 1uF, Library:C0603, symbol Library:CL10A105KB8NNNC Capacitor 1uF
- added Q14, Q16, Q18, Q20, Q21, Q22: (no value), Library:WDFN-5_L3.1-W3.1-P0.65-BL_1, symbol Library:40N06D MOSFET N-Channel 40A
- added R68: 1kΩ, Library:R0603, symbol Library:0603WAF1001T5E Resistor 1kΩ
- added R72: 10kΩ, Library:R0603, symbol Library:0603WAF1002T5E Resistor 10kΩ
- added R77, R81, R90, R92, R93, R94: 4.7Ω, Library:R0603, symbol Library:0603WAF470KT5E Resistor 4.7Ω
- added U42: (no value), Library:ESSOP-10_L4.9-W3.9-P1.0-LS6.0-TL-EP, symbol Library:CH224K USB PD 20V sink controller
- added U46, U47: (no value), Library:SOIC-8_L4.9-W3.9-P1.27-LS6.0-BL, symbol Library:MX5014S High side/Low side MOSFET gate driver
- U19: now fitted
Connections:
- net VBATTERY_MID_DIODE is gone; now on net VANY: D12.1 (-)
- net VBUS_MID_DIODE is gone; now on net VANY: D14.1 (-)
- net +Probe-6: now also U16.7 (IN±2); no longer U16.6 (IN+2)
- net +Probe-7: now also U16.17 (IN+4); no longer U16.14 (IN±3)
- net +Probe-8: now also U16.14 (IN±3); no longer U16.17 (IN+4)
- net -Probe-6: now also U16.6 (IN+2); no longer U16.7 (IN±2)
- net -Probe-7: now also U16.18 (IN±4); no longer U16.15 (IN+3)
- net -Probe-8: now also U16.15 (IN+3); no longer U16.18 (IN±4)
- net BATTERY_CURRENT: now also U1.6 (IO6), U16.13 (OUT3); no longer U1.5 (IO5), U16.19 (OUT4)
- net CAN_RX: now also U1.23 (IO21); no longer U1.22 (IO14)
- net CAN_TX: now also U1.22 (IO14); no longer U1.23 (IO21)
- net CC1: now also U42.7 (CC1)
- net CC2: now also U42.6 (CC2)
- net CONNECT_BATTERY: now also U47.2 (Input)
- net CONNECT_VBUS: now also U46.2 (Input)
- net GND: now also C29.1, C55.1, C56.1, U42.11 (GND), U42.3 (CFG3), U42.9 (CFG1), U46.4 (GND), U47.4 (GND)
- net GUEST_USB_D+: now also U42.4 (DP)
- net GUEST_USB_D-: now also U42.5 (DM)
- net VBATTERY: now also R8.2 (Shunt-2), Q18.5 (D), Q21.5 (D); no longer U19.6, U19.7, U19.8
- net VBUS: now also R7.2 (Shunt-2), Q14.5 (D), R68.1, R72.1; no longer USB0.A4B9 (VBUS), USB0.B4A9 (VBUS)
- net VBUS_CURRENT: now also U1.5 (IO5), U16.19 (OUT4); no longer U1.6 (IO6), U16.13 (OUT3)
- net VCC: now also Q16.5 (D), Q20.5 (D), Q22.5 (D); no longer R7.2 (Shunt-2), R8.2 (Shunt-2)
- net Buck-VIN renamed VANY
- net VANY: now also C55.2, C56.2, U46.1 (V+), U47.1 (V+)
- net VBATTERY_PROBE renamed VBATTERY_PINS
- net VBATTERY_PINS: now also U19.6, U19.7, U19.8
- net VBUS_PROBE renamed VBUS_PINS
- net VBUS_PINS: now also USB0.A4B9 (VBUS), USB0.B4A9 (VBUS)
- new net: R77.1, R81.1, U46.5 (Gate)
- new net: R90.1, R92.1, R93.1, R94.1, U47.5 (Gate)
- new net Gate1-vbattery: Q18.4 (G), R90.2
- new net Gate1-vbus: Q14.4 (G), R81.2
- new net Gate2-vbattery: Q20.4 (G), R92.2
- new net Gate2-vbus: Q16.4 (G), R77.2
- new net Gate3-vbattery: Q21.4 (G), R93.2
- new net Gate4-vbattery: Q22.4 (G), R94.2
- new net PD-VBUS-DETECT: R72.2, U42.8 (VBUS)
- new net PD-VDD: C29.2, R68.2, U42.1 (VDD), U42.2 (CFG2)
- new net Source-vbattery: Q18.1 (S), Q18.2 (S), Q18.3 (S), Q20.1 (S), Q20.2 (S), Q20.3 (S), Q21.1 (S), Q21.2 (S), Q21.3 (S), Q22.1 (S), Q22.2 (S), Q22.3 (S), U47.3 (Source)
- new net Source-vbus: Q14.1 (S), Q14.2 (S), Q14.3 (S), Q16.1 (S), Q16.2 (S), Q16.3 (S), U46.3 (Source)
- no-connect marks 62 -> 69
Other:
- removed sheet back-to-back-mosfets
- removed sheet back-to-back-mosfets1
- removed sheet back-to-back-mosfets2
- note added: "Hex Master USB Hub Controller"
- note added: "OR-ing diodes gives power to VANY from any of the VBATTERY or VBUS sources. We use this to 1. turn on the esp32 microcontroller and 2. power the gate drivers for the VCC switches."
- note added: "Power management"
- note removed: "20nF capacitor requests 20V"
- note removed: "5V and 3V3 power regulator and filtering"
- note removed: "Main power comes from the VCC bus, but we have diodes to wakeup the microcontroller, which turns on the VCC line. There's a single diode from VCC so we prefer VCC, double diodes on the input VBUS and VBATTERY."
- moved on the sheet: C1, C10, C11, C12, C13, C16, C17, C18, C2, C20, C21, C22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
