File: symbols-and-footprints/Library.kicad_blocks/back-to-back-mosfets.kicad_block/back-to-back-mosfets.kicad_pcb (KiCad board)
At the start: 4 copper layers, 6 parts

Commit message: Design block experimentation.
Parts:
- C29, C49, Q5, Q6, R36, U12: moved to B.Cu
- moved R36 220.4 mm to (87.4, 111.5), turned to 180 degrees
- moved C49 220.0 mm to (87.4, 109.8)
- moved Q6 219.9 mm to (87.6, 114.9), turned to -90 degrees
- moved U12 219.1 mm to (85.0, 112.0), turned to 0 degrees
- moved Q5 218.3 mm to (82.1, 114.8), turned to 90 degrees
- moved C29 217.4 mm to (82.7, 111.6), turned to 0 degrees
Connections:
- net /VCC_PROBE renamed /VBUS_PROBE
- net Net-(Q5-D) renamed /back-to-back-mosfets/Mid-MOSFETSx
- net Net-(Q5-G) renamed /back-to-back-mosfets/GATE2x
- net Net-(Q6-G) renamed /back-to-back-mosfets/GATE1x
Routing:
- net VBUS: track 0.00 -> 6.97 mm
- net /VBUS_PROBE: track 0.00 -> 6.62 mm
- net /back-to-back-mosfets/GATE1x: track 0.00 -> 6.61 mm
- net GND: track 0.00 -> 4.47 mm, vias 0 -> 4
- net /back-to-back-mosfets/GATE2x: track 0.00 -> 4.28 mm
- net CONNECT_VBUS: track 0.00 -> 1.79 mm
